File: HW/LoRa_TM/LoRa_TM.kicad_pcb (KiCad board)
At the start: 2 copper layers, 39 parts, among them J1 USB_C_USB2.0_14P, J2 SMA, J3 GH 1.25mm 6P, J4 GH 1.25mm 6P, U1 STM32U375CGT6, U2 USBLC6-2SC6, U3 TPS62842DGR, U4 E22-900T33S, Y1 16MHz

Commit message: PCB Done
Parts:
- removed C10: 4.7uF, Capacitor_SMD:C_0603_1608Metric
- removed C11: 10uF, Capacitor_SMD:C_0603_1608Metric
- removed C8, C9: 10pF, Capacitor_SMD:C_0603_1608Metric
- removed D5: Red, LED_SMD:LED_0603_1608Metric
- removed J4: GH 1.25mm 6P, JST_GH:JST_GH_SM06B-GHS-TB_06x1.25mm_Angled
- removed R4: 10k, Resistor_SMD:R_0603_1608Metric
- removed R6, R7, R8: 120, Resistor_SMD:R_0603_1608Metric
- removed Y1: 16MHz, Crystal:Crystal_SMD_Abracon_ABM8G-4Pin_3.2x2.5mm
- added J5: GH 1.25mm 6P, JST_GH:JST_GH_SM06B-GHS-TB_06x1.25mm_Angled, F.Cu at (107.3, 73.6)
- added R14: 0, Resistor_SMD:R_0603_1608Metric, B.Cu at (109.3, 85.7)
- added R15: 10k, Resistor_SMD:R_0603_1608Metric, B.Cu at (93.1, 94.2)
- C1, C2, C4, C5, D1, L1, R1, R10, R2: moved to B.Cu
- C3: value 100nF -> 10nF; moved to B.Cu
- C6: value 100nF -> 10uF; moved to B.Cu
- C7: value 1ouF -> 4.7uF; moved to B.Cu
- J1: value USB_C_USB2.0_14P -> GH 1.25mm 10P; footprint Connector_USB:USB_C_Receptacle_GCT_USB4110 -> JST_GH:JST_GH_SM10B-GHS-TB_10x1.25mm_Angled; moved to B.Cu
- J2: value SMA -> USB_C_USB2.0_14P; footprint Connector_Coaxial:SMA_Amphenol_132289_EdgeMount -> Connector_USB:USB_C_Receptacle_GCT_USB4110
- J3: value GH 1.25mm 6P -> SMA; footprint JST_GH:JST_GH_SM06B-GHS-TB_06x1.25mm_Angled -> SMA:SMA_EdgeMount
- R11, R13: value 10k -> 120
- R12: value 52k3 -> 120
- R3: value 1k5 -> 10k; moved to B.Cu
- R5: value 120 -> 52k3; moved to B.Cu
- R9: value 120 -> 10k; moved to B.Cu
- U1: value STM32U375CGT6 -> STM32F042F4P6TR; footprint STM32U375CGT6:LQFP48_STM -> STM32F042F4P6TR:TSSOP20; moved to B.Cu
- U2: value USBLC6-2SC6 -> TPS62842DGR; footprint Package_TO_SOT_SMD:SOT-23-6 -> Package_SO:HVSSOP-8-1EP_3x3mm_P0.65mm_EP1.57x1.89mm; moved to B.Cu
- U3: value TPS62842DGR -> USBLC6-2SC6; footprint Package_SO:HVSSOP-8-1EP_3x3mm_P0.65mm_EP1.57x1.89mm -> Package_TO_SOT_SMD:SOT-23-6; moved to B.Cu
- moved J3 135.3 mm to (92.9, 125.1), turned to -90 degrees
- moved D2 125.2 mm to (106.6, 125.7), turned to 90 degrees
- moved R11 121.6 mm to (108.1, 125.7), turned to 90 degrees
- moved D3 121.3 mm to (103.1, 125.7), turned to 90 degrees
- moved R12 117.6 mm to (104.6, 125.7), turned to 90 degrees
- moved U4 117.4 mm to (100.0, 100.0)
- moved D4 117.3 mm to (99.6, 125.7), turned to 90 degrees
- moved R13 113.6 mm to (101.1, 125.7), turned to 90 degrees
- moved C3 98.0 mm to (103.0, 86.5), turned to -90 degrees
- moved C1 96.8 mm to (108.3, 72.9)
- moved C5 95.9 mm to (104.6, 86.5), turned to -90 degrees
- moved U1 95.9 mm to (98.1, 86.5), turned to 180 degrees
- moved C6 94.4 mm to (110.8, 77.5), turned to 90 degrees
- moved R10 93.3 mm to (93.1, 99.2)
- moved R9 93.3 mm to (93.1, 96.7)
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Connections:
- C1 pad 1: Net-(U1-VCAP) -> +5V
- C3 pad 2: GNDA -> GND
- C5 pad 2: GNDA -> GND
- J3 pad 1: +5V -> Net-(J3-In)
- J3 pad 2: /USART1_RX -> GND
- L1 pad 1: Net-(U3-SW) -> Net-(U2-SW)
- R1 pad 1: Net-(J1-CC1) -> Net-(J2-CC1)
- R10 pad 1: /LoRa_M1 -> /LoRa_M0
- R11 pad 1: /LoRa_M0 -> Net-(D2-K)
- R12 pad 1: GND -> Net-(D3-K)
- R12 pad 2: Net-(U3-VSET) -> GND
- R13 pad 1: +3.3V -> Net-(D4-K)
- R13 pad 2: /USART1_RX -> GND
- R2 pad 1: Net-(J1-CC2) -> Net-(J2-CC2)
- R3 pad 1: +3.3V -> GND
- R3 pad 2: /USB_D+ -> /BOOT0
- R5 pad 1: Net-(D2-K) -> GND
- R5 pad 2: GND -> Net-(U2-VSET)
- R9 pad 1: Net-(C8-Pad1) -> /LoRa_M1
- R9 pad 2: /OSC_OUT -> GND
- U1 pad 1: +3.3V -> /BOOT0
- U1 pad 10: /LoRa_AUX -> /LED_TX
- U1 pad 11: /LoRa_M0 -> /LED_RX
- U1 pad 12: /LoRa_M1 -> /LED_ON
- U1 pad 14: unconnected-(U1-PA4-Pad14) -> /LoRa_AUX
- U1 pad 15: /LoRa_RX -> GND
- U1 pad 16: unconnected-(U1-PA6-Pad16) -> +3.3V
- U1 pad 17: /LoRa_TX -> /USB_D-
- U1 pad 18: unconnected-(U1-PB0-Pad18) -> /USB_D+
- U1 pad 19: unconnected-(U1-PB1-Pad19) -> /SWDIO
- U1 pad 2: unconnected-(U1-PC13-Pad2) -> /LoRa_M0
- U1 pad 20: unconnected-(U1-PB2-Pad20) -> /SWCLK
- U1 pad 3: unconnected-(U1-PC14-OSC32_IN-Pad3) -> /LoRa_M1
- U1 pad 4: unconnected-(U1-PC15-OSC32_OUT-Pad4) -> /NRST
- U1 pad 5: /OSC_IN -> +3.3V
- U1 pad 6: /OSC_OUT -> unconnected-(U1-PA0-Pad6)
- U1 pad 7: /NRST -> unconnected-(U1-PA1-Pad7)
- U1 pad 8: GNDA -> /LoRa_RX
- U1 pad 9: +3.3V -> /LoRa_TX
- U2 pad 1: /USB_CONN_D- -> +3.3V
- U2 pad 2: GND -> Net-(U2-SW)
- U2 pad 3: /USB_CONN_D+ -> GND
- U2 pad 4: /USB_D+ -> Net-(U2-VSET)
- U2 pad 5: VBUS -> +5V
- U2 pad 6: /USB_D- -> +5V
- U3 pad 1: +3.3V -> /USB_D-
- U3 pad 2: Net-(U3-SW) -> GND
- U3 pad 3: GND -> /USB_CONN_D-
- U3 pad 4: Net-(U3-VSET) -> /USB_CONN_D+
- U3 pad 5: +5V -> VBUS
- U3 pad 6: +5V -> /USB_D+
- U4 pad 11: Net-(J2-In) -> Net-(J3-In)
- U4 pad 23: GND -> Net-(R14-Pad2)
- U4 pad 4: /LoRa_RX -> /LoRa_TX
- U4 pad 5: /LoRa_TX -> /LoRa_RX
Routing:
- net +5V: track 0.00 -> 42.2 mm, vias 0 -> 2
- net /LED_RX: track 0.00 -> 40.4 mm, vias 0 -> 1
- net /LED_ON: track 0.00 -> 39.7 mm, vias 0 -> 1
- net /LED_TX: track 0.00 -> 38.7 mm, vias 0 -> 1
- net /LoRa_RX: track 0.00 -> 38.3 mm, vias 0 -> 2
- net /LoRa_M0: track 0.00 -> 36.5 mm, vias 0 -> 2
- net /LoRa_TX: track 0.00 -> 35.2 mm, vias 0 -> 1
- net /LoRa_M1: track 0.00 -> 34.3 mm, vias 0 -> 2
- net /LoRa_AUX: track 0.00 -> 22.7 mm, vias 0 -> 1
- net +3.3V: track 0.00 -> 18.1 mm, vias 0 -> 5
- net /NRST: track 0.00 -> 17.5 mm, vias 0 -> 2
- net GND: track 0.00 -> 15.9 mm, vias 0 -> 16
- net /BOOT0: track 0.00 -> 15.7 mm, vias 0 -> 2
- net VBUS: track 0.00 -> 15.4 mm, vias 0 -> 2
- net /SWDIO: track 0.00 -> 15.2 mm, vias 0 -> 2
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- added copper zone on In2.Cu, net +3.3V
- added copper zone on B.Cu, net GND
- added copper zone on F.Cu, net GND
- added copper zone on In1.Cu, net GND
- added copper zone on In2.Cu, net GND
Other:
- board outline added: 28 x 58 mm
- copper layers 2 -> 4
- board text added: "- [ ] 433 MHz - [ ] 900 MHz"
- board text added: "For E22"
- board text added: "LoRa TM NARAE INHA University Rev 2.0"
- board text added: "ON"
- board text added: "RX"
- board text added: "Stack Up : JLC04161H-7628"
- board text added: "TX"
