File: HW/LoRa_TM/LoRa_TM.kicad_sch (KiCad schematic)
At the start: 39 parts, among them J1 USB_C_USB2.0_14P, J2 SMA, J3 GH 1.25mm 6P, J4 GH 1.25mm 6P, U1 STM32U375CGT6, U2 USBLC6-2SC6, U3 TPS62842DGR, U4 E22-900T33S, Y1 16MHz

Commit message: stm32u375 update
Parts:
- added R13: 0, Resistor_SMD:R_0603_1608Metric, symbol Device:R_Small_US
- C9: renamed from C7; value 1ouF -> 10uF
- renumbered C8 to C7, C9 to C8, R13 to R14, R4 to R3, R3 to R4
Connections:
- net GND: now also R13.1; no longer U4.23 (GND)
- new net: R13.2, U4.23 (GND)
Other:
- moved on the sheet: J2, R10, R11, U4

Commit message: PCB Done
Parts:
- removed C1: 4.7uF, Capacitor_SMD:C_0603_1608Metric, symbol Device:C_Small
- removed C2: 100nF, Capacitor_SMD:C_0603_1608Metric, symbol Device:C_Small
- removed C7, C8: 10pF, Capacitor_SMD:C_0603_1608Metric, symbol Device:C_Small
- removed D5: Red, LED_SMD:LED_0603_1608Metric, symbol Device:LED_Small
- removed R4: 1k5, Resistor_SMD:R_0603_1608Metric, symbol Device:R_Small_US
- removed R8, R9: 120, Resistor_SMD:R_0603_1608Metric, symbol Device:R_Small_US
- removed U1: STM32U375CGT6, LQFP48_STM, symbol STM32U375CGT6:STM32U375CGT6
- removed Y1: 16MHz, Crystal:Crystal_SMD_Abracon_ABM8G-4Pin_3.2x2.5mm, symbol Device:Crystal_GND24_Small
- added U1: STM32F042F4P6TR, STM32F042F4P6TR:TSSOP20, symbol STM32F042F4P6TR:STM32F042F4P6TR
- C1: renamed from C10; LCSC C307423 -> C1705
- C2: renamed from C4; LCSC C1525 -> C1590
- C3: value 100nF -> 10nF; LCSC C1525 -> C1589
- C4: renamed from C6; LCSC C1525 -> C1590
- C5: LCSC C1525 -> C1592
- C6: renamed from C11; LCSC C307415 -> C1691
- C7: renamed from C9; value 10uF -> 4.7uF; LCSC C1525 -> C1705
- D1: LCSC C22624 -> C64885
- D2, D3, D4: LCSC C130719 -> C2286
- J1: renamed from J4; value GH 1.25mm 6P -> GH 1.25mm 10P; footprint JST_GH:JST_GH_SM06B-GHS-TB_06x1.25mm_Angled -> JST_GH:JST_GH_SM10B-GHS-TB_10x1.25mm_Angled; symbol Connector_Generic:Conn_01x06 -> Connector_Generic:Conn_01x10; LCSC C133065 -> C2683602
- J3: renamed from J2; footprint Connector_Coaxial:SMA_Amphenol_132289_EdgeMount -> SMA:SMA_EdgeMount
- J5: renamed from J3; LCSC C133065 -> C133065
- L1: LCSC C114768 -> (none)
- R1, R2: LCSC C25905 -> C14677
- R10: renamed from R11; LCSC C25079 -> C15401
- R11: renamed from R5; LCSC C25079 -> C22787
- R12: renamed from R6; LCSC C25079 -> C22787
- R13: renamed from R7; LCSC C25079 -> C22787
- R14: renamed from R13; LCSC C25079 -> C15402
- R15: renamed from R14; LCSC C25531 -> C15401
- R3: LCSC C25079 -> C15401
- R5: renamed from R12; LCSC C2998050 -> (none)
- R9: renamed from R10; LCSC C25079 -> C15401
- U2: renamed from U3; LCSC (none) -> C2873354
- renumbered J1 to J2, U2 to U3
Connections:
- net USART1_RX is gone; now on net LoRa_RX: J5.2 (Pin_2), R15.2
- net USART1_TX is gone; now on net LoRa_TX: J5.3 (Pin_3)
- net +3.3V: now also J1.2 (Pin_2), U1.16 (VDD), U1.5 (VDDA)
- net BOOT0: now also J1.6 (Pin_6), U1.1 (PB8-BOOT0); no longer J1.5 (Pin_5)
- net GND: now also C3.2, C5.2, J1.10 (Pin_10), U1.15 (VSS); no longer J1.6 (Pin_6)
- net GNDA: no longer C3.2, C5.2
- net LED_ON: now also U1.12 (PA6)
- net LED_RX: now also U1.11 (PA5)
- net LED_TX: now also U1.10 (PA4)
- net LoRa_AUX: now also J1.7 (Pin_7), U1.14 (PB1)
- net LoRa_M0: now also J1.9 (Pin_9), U1.2 (PF0-OSC_IN)
- net LoRa_M1: now also J1.8 (Pin_8), U1.3 (PF1-OSC_OUT)
- net LoRa_RX: now also U4.5 (RXD), U1.8 (PA2); no longer U4.4 (TXD)
- net LoRa_TX: now also U4.4 (TXD), U1.9 (PA3); no longer U4.5 (RXD)
- net NRST: now also J1.5 (Pin_5), U1.4 (NRST); no longer J1.4 (Pin_4)
- net SWCLK: now also J1.4 (Pin_4), U1.20 (PA14); no longer J1.3 (Pin_3)
- net SWDIO: now also J1.3 (Pin_3), U1.19 (PA13); no longer J1.2 (Pin_2)
- net USB_CONN_D+: now also U3.4 (I/O2); no longer U3.3 (I/O2)
- net USB_CONN_D-: now also U3.3 (I/O2); no longer U3.1 (I/O1)
- net USB_D+: now also U3.6 (I/O1), U1.18 (PA10/PA12); no longer U3.4 (I/O2)
- net USB_D-: now also U3.1 (I/O1), U1.17 (PA9/PA11); no longer U3.6 (I/O1)
- net USART1_CTS: no longer names the net of J5.4 (Pin_4)
- net USART1_RTS: no longer names the net of J5.5 (Pin_5)
- no-connect marks 19 -> 7
Other:
- note added: "AUX : PA0 TXD : PA3 (USART2_RX) RXD : PA2 (USART2_TX) M1 : PA2 M0 : PA1"
- note added: "STM32F042F4 is embedded pull up R"
- note added: "USART2_RX"
- note added: "USART2_TX"
- note removed: "AUX : PA0 TXD : PA5 (USART3_RX) RXD : PA7 (USART3_TX) M1 : PA2 M0 : PA1"
- moved on the sheet: C1, C2, C3, C4, C5, C6, C7, D2, D3, D4, L1, R11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

Commit message: Schematic update
Other:
- title: LoRa TM (900MHz) -> LoRa TM
Changed lines of the file:
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@@
 	(paper "A4")
 	(title_block
-		(title "LoRa TM (900MHz)")
-		(date "2025-06-13")
-		(rev "v1.0")
+		(title "LoRa TM")
+		(date "2025-06-18")
+		(rev "v2.0")
 		(company "NARAE")
 		(comment 1 "INHA Univ. Areo-modelling Club")
